Commit message: Imported upstream version '2.0.0' of 'upstream'

File: rb1_base_description/urdf/bases/rb1_base.gazebo.xacro (robot description, xacro)
@@ -1,47 +1,53 @@
 <?xml version="1.0"?>
-<robot xmlns:xacro="http://ros.org/wiki/xacro">
-  <!-- ros control plugin -->
-  <!-- xacro:macro name="ros_control">
-    <gazebo>
+<robot xmlns:xacro="http://www.ros.org/wiki/xacro">
+	<!-- DIFFERENCIAL DRIVE GAZEBO PLUGIN -->
+	<xacro:macro name="gazebo_differencial_drive">
+		<gazebo>
+			<plugin name="differential_drive_controller" filename="libgazebo_ros_diff_drive.so">
+				<!--alwaysOn>true</alwaysOn-->
+				<updateRate>50.0</updateRate>
+				<leftJoint>$(prefix_frame)rb1_a_left_wheel_joint</leftJoint>
+				<rightJoint>$(prefix_frame)rb1_a_right_wheel_joint</rightJoint>
+				<!--leftJoint>joint_right_wheel</leftJoint>
+				<rightJoint>joint_left_wheel</rightJoint-->
+				<!-- For V0 0.365 -->
+				<!-- wheelSeparation>0.365</wheelSeparation -->
+				<wheelSeparation>0.433</wheelSeparation>
+				<wheelDiameter>0.1524</wheelDiameter>
+				<commandTopic>rb1/cmd_vel</commandTopic>
+				<odometryTopic>odom</odometryTopic>
+				<odometryFrame>$(prefix_frame)odom</odometryFrame>
+				<robotBaseFrame>$(prefix_frame)base_link</robotBaseFrame>
+				<!-- robotNamespace></robotNamespace -->
+				<rosDebugLevel>na</rosDebugLevel>
+				<publishWheelTF>false</publishWheelTF>
+				<publishWheelJointState>true</publishWheelJointState>
+				<wheelAcceleration>0</wheelAcceleration>
+				<wheelTorque>5</wheelTorque>
+				<!-- odometrySource>encoder</odometrySource -->
+				<odometrySource>encoder</odometrySource>
+				<legacyMode>false</legacyMode>
+				<publishTf>1</publishTf>
+			</plugin>
+		</gazebo>
+	</xacro:macro>
+	<xacro:macro name="ros_control" params="prefix_frame prefix_topic">
+	   <gazebo>
       <plugin name="ros_control" filename="libgazebo_ros_control.so">
-        <robotNamespace>/rb1</robotNamespace>
+        <!--robotNamespace>/rb1</robotNamespace-->
         <robotParam>robot_description</robotParam>
         <controlPeriod>0.001</controlPeriod>
 	    <robotSimType>gazebo_ros_control/DefaultRobotHWSim</robotSimType>
       </plugin>
-    </gazebo>
-	</xacro:macro -->
-	<!-- differential drive plugin -->
-	<xacro:macro name="diff_drive">
-    <gazebo>
-	<plugin name="differential_drive_controller" filename="libgazebo_ros_diff_drive.so">
-	    <alwaysOn>true</alwaysOn>
-        <updateRate>50.0</updateRate>
-        <!-- leftJoint>joint_left_wheel</leftJoint>
-        <rightJoint>joint_right_wheel</rightJoint -->
-        <leftJoint>joint_right_wheel</leftJoint>
-        <rightJoint>joint_left_wheel</rightJoint>
-		<!-- For V0 0.365 -->
-        <!-- wheelSeparation>0.365</wheelSeparation -->
-        <wheelSeparation>0.433</wheelSeparation>
-        <wheelDiameter>0.1524</wheelDiameter>
-        <commandTopic>/rb1/cmd_vel</commandTopic>
-        <odometryTopic>odom</odometryTopic>
-        <odometryFrame>odom</odometryFrame>
-        <robotBaseFrame>base_footprint</robotBaseFrame>
-        <!-- robotNamespace></robotNamespace -->
-        <rosDebugLevel>na</rosDebugLevel>
-        <publishWheelTF>false</publishWheelTF>
-        <publishWheelJointState>false</publishWheelJointState>
-        <wheelAcceleration>0</wheelAcceleration>
-        <wheelTorque>5</wheelTorque>
-        <!-- odometrySource>encoder</odometrySource -->
-        <odometrySource>world</odometrySource>
-        <publishTf>1</publishTf>
-	</plugin>
+   </gazebo>
+   </xacro:macro>
+	<gazebo reference="base_footprint">
+		<material>Gazebo/Green</material>
 	</gazebo>
-    </xacro:macro>
-  <gazebo reference="base_footprint">
-    <material>Gazebo/Green</material>
-  </gazebo>
+	<gazebo reference="base_link">
+		<material>Gazebo/Grey</material>
+	</gazebo>
+	<gazebo reference="front_cover_link">
+		<material>Gazebo/Black</material>
+	</gazebo>
 </robot>

File: rb1_base_description/urdf/bases/rb1_base.urdf.xacro (robot description, xacro)
@@ -1,6 +1,5 @@
 <?xml version="1.0"?>
 <robot name="rb1_base" xmlns:xacro="http://www.ros.org/wiki/xacro">
-  <!-- xacro:include filename="$(find rb1_base_description)/urdf/bases/rb1_base.gazebo.xacro" / -->
-  <xacro:macro name="rb1_base" params="name publish_bf hq">
+  <xacro:macro name="rb1_base" params="prefix publish_bf hq">
   <!-- Robot mechanical and motor parameters -->
   <xacro:property name="PI" value="3.1415926535897931"/>
@@ -8,5 +7,5 @@
   <!-- BASE FOOTPRINT -->
   <xacro:if value="${publish_bf}">
-    <link name="base_footprint">
+    <link name="${prefix}base_footprint">
       <visual>
           <origin xyz="0 0 0" rpy="0 0 0" />
@@ -16,16 +15,16 @@
       </visual>
     </link>
-    <joint name="base_footprint_joint" type="fixed">
+    <joint name="${prefix}base_footprint_joint" type="fixed">
        <origin xyz="0 0 ${wheel_radius - wheel_offset_z}" rpy="0 0 0" />
-      <parent link="base_footprint"/>
-      <child link="base_link" />
+      <parent link="${prefix}base_footprint"/>
+      <child link="${prefix}base_link" />
     </joint>
   </xacro:if>
   <!-- BASE_LINK -->
-  <link name="base_link">
+  <link name="${prefix}base_link">
     <inertial>
       <mass value="25.0" />
       <origin xyz="0 0 0" />
-      <inertia  ixx="0.007" ixy="0.0"  ixz="0.0"  iyy="0.007"  iyz="0.0"  izz="0.78" />
+      <inertia  ixx="0.605" ixy="0.0"  ixz="0.0"  iyy="0.5435"  iyz="0.0"  izz="0.981" />
     </inertial>
     <visual>
@@ -33,5 +32,5 @@
        <xacro:if value="${hq}">
        <geometry>
-	     <mesh filename="package://rb1_base_description/meshes/bases/rb1v2_base.dae"/>
+         <mesh filename="package://rb1_base_description/meshes/bases/rb1v2_base.dae"/>
        </geometry>
        </xacro:if>
@@ -52,11 +51,11 @@
     </collision>
   </link>
-  <joint name="front_cover_joint" type="fixed">
+  <joint name="${prefix}front_cover_joint" type="fixed">
      <origin xyz="0.220 0.0 0.004" rpy="0 0 0 " />
-     <parent link="base_link"/>
-     <child link="front_cover_link" />
+     <parent link="${prefix}base_link"/>
+     <child link="${prefix}front_cover_link" />
   </joint>
   <!-- FRONT COVER -->
-  <link name="front_cover_link">
+  <link name="${prefix}front_cover_link">
     <inertial>
       <mass value="0.25" />
@@ -88,11 +87,11 @@
   </link>
   <!-- DOCKING CONTACTS -->
-  <joint name="base_docking_joint" type="fixed">
+  <joint name="${prefix}base_docking_joint" type="fixed">
      <origin xyz="0.030 0.000 0.068" rpy="0 0 0 " />
-     <parent link="front_cover_link"/>
-     <child link="base_docking_contact" />
+     <parent link="${prefix}front_cover_link"/>
+     <child link="${prefix}base_docking_contact" />
   </joint>
   <!-- FRONT COVER -->
-  <link name="base_docking_contact" />
+  <link name="${prefix}base_docking_contact" />
   </xacro:macro>
 </robot>

File: rb1_base_description/urdf/bases/rb1_base_v0.urdf.xacro (robot description, xacro)
@@ -1,6 +1,5 @@
 <?xml version="1.0"?>
 <robot name="rb1_base" xmlns:xacro="http://www.ros.org/wiki/xacro">
-  <xacro:include filename="$(find rb1_base_description)/urdf/bases/rb1_base.gazebo.xacro" />
-  <xacro:macro name="rb1_base" params="name publish_bf hq">
+  <xacro:macro name="rb1_base_v0" params="prefix publish_bf hq">
   <!-- Robot mechanical and motor parameters -->
   <xacro:property name="PI" value="3.1415926535897931"/>
@@ -8,5 +7,5 @@
   <!-- BASE FOOTPRINT -->
   <xacro:if value="${publish_bf}">
-    <link name="base_footprint">
+    <link name="${prefix}base_footprint">
       <visual>
           <origin xyz="0 0 0" rpy="0 0 0" />
@@ -16,16 +15,16 @@
       </visual>
     </link>
-    <joint name="base_footprint_joint" type="fixed">
+    <joint name="${prefix}base_footprint_joint" type="fixed">
        <origin xyz="0 0 ${wheel_radius - wheel_offset_z}" rpy="0 0 0" />
-      <parent link="base_footprint"/>
-      <child link="base_link" />
+      <parent link="${prefix}base_footprint"/>
+      <child link="${prefix}base_link" />
     </joint>
   </xacro:if>
   <!-- BASE_LINK -->
-  <link name="base_link">
+  <link name="${prefix}base_link">
     <inertial>
       <mass value="25.0" />
       <origin xyz="0 0 0" />
-      <inertia  ixx="1.0" ixy="0.0"  ixz="0.0"  iyy="1.0"  iyz="0.0"  izz="1.0" />
+      <inertia  ixx="0.605" ixy="0.0"  ixz="0.0"  iyy="0.5435"  iyz="0.0"  izz="0.981" />
     </inertial>
     <visual>
@@ -33,10 +32,10 @@
        <xacro:if value="${hq}">
        <geometry>
-	     <mesh filename="package://rb1_base_description/meshes/bases/rb1_base_v0.dae"/>
+         <mesh filename="package://rb1_base_description/meshes/bases/rb1v0_base.dae"/>
        </geometry>
        </xacro:if>
        <xacro:unless value="${hq}">
        <geometry>
-       <mesh filename="package://rb1_base_description/meshes/bases/rb1_base_v0.stl"/>
+       <mesh filename="package://rb1_base_description/meshes/bases/rb1v0_base.stl"/>
        </geometry>
        </xacro:unless>
@@ -48,5 +47,5 @@
        <origin xyz="0 0 0" rpy="0 0 0 " />
        <geometry>
-         <mesh filename="package://rb1_base_description/meshes/bases/rb1_base_v0.dae"/>
+         <mesh filename="package://rb1_base_description/meshes/bases/rb1v0_base.dae"/>
        </geometry>
     </collision>

File: rb1_base_description/urdf/bases/rb1_base_v1.urdf.xacro (robot description, xacro)
@@ -1,6 +1,5 @@
 <?xml version="1.0"?>
 <robot name="rb1_base" xmlns:xacro="http://www.ros.org/wiki/xacro">
-  <xacro:include filename="$(find rb1_base_description)/urdf/bases/rb1_base.gazebo.xacro" />
-  <xacro:macro name="rb1_base" params="name publish_bf hq">
+  <xacro:macro name="rb1_base_v1" params="prefix publish_bf hq">
   <!-- Robot mechanical and motor parameters -->
   <xacro:property name="PI" value="3.1415926535897931"/>
@@ -8,5 +7,5 @@
   <!-- BASE FOOTPRINT -->
   <xacro:if value="${publish_bf}">
-    <link name="base_footprint">
+    <link name="${prefix}base_footprint">
       <visual>
           <origin xyz="0 0 0" rpy="0 0 0" />
@@ -16,16 +15,16 @@
       </visual>
     </link>
-    <joint name="base_footprint_joint" type="fixed">
+    <joint name="${prefix}base_footprint_joint" type="fixed">
        <origin xyz="0 0 ${wheel_radius - wheel_offset_z}" rpy="0 0 0" />
-      <parent link="base_footprint"/>
-      <child link="base_link" />
+      <parent link="${prefix}base_footprint"/>
+      <child link="${prefix}base_link" />
     </joint>
   </xacro:if>
   <!-- BASE_LINK -->
-  <link name="base_link">
+  <link name="${prefix}base_link">
     <inertial>
       <mass value="25.0" />
       <origin xyz="0 0 0" />
-      <inertia  ixx="0.007" ixy="0.0"  ixz="0.0"  iyy="0.007"  iyz="0.0"  izz="0.78" />
+      <inertia  ixx="0.605" ixy="0.0"  ixz="0.0"  iyy="0.5435"  iyz="0.0"  izz="0.981" />
     </inertial>
     <visual>
@@ -33,10 +32,10 @@
        <xacro:if value="${hq}">
        <geometry>
-	     <mesh filename="package://rb1_base_description/meshes/bases/rb1_base.dae"/>
+	     <mesh filename="package://rb1_base_description/meshes/bases/rb1v1_base.dae"/>
        </geometry>
        </xacro:if>
        <xacro:unless value="${hq}">
        <geometry>
-       <mesh filename="package://rb1_base_description/meshes/bases/rb1_base.stl"/>
+       <mesh filename="package://rb1_base_description/meshes/bases/rb1v1_base.stl"/>
        </geometry>
        </xacro:unless>
@@ -48,5 +47,5 @@
        <origin xyz="0 0 0" rpy="0 0 0 " />
        <geometry>
-         <mesh filename="package://rb1_base_description/meshes/bases/rb1_base.dae"/>
+         <mesh filename="package://rb1_base_description/meshes/bases/rb1v1_base.dae"/>
        </geometry>
     </collision>

File: rb1_base_description/urdf/wheels/omni_wheel.urdf.xacro (robot description, xacro)
@@ -3,24 +3,25 @@
   <xacro:property name="M_PI" value="3.1415926535897931" />
   <!-- Wheels -->
-  <property name="omni_wheel_radius" value="0.051" />
-  <property name="omni_wheel_height" value="0.040" />
-  <property name="omni_wheel_mass" value="0.3" /> <!-- in kg-->
+  <xacro:property name="omni_wheel_radius" value="0.051" />
+  <xacro:property name="omni_wheel_height" value="0.040" />
+  <xacro:property name="omni_wheel_mass" value="0.3" /> <!-- in kg-->
   <xacro:macro name="cylinder_inertia" params="m r h">
     <inertia  ixx="${m*(3*r*r+h*h)/12}" ixy = "0" ixz = "0"
               iyy="${m*(3*r*r+h*h)/12}" iyz = "0"
-              izz="${m*r*r/2}" />
+              izz="${m*r*r/2}"
+     />
   </xacro:macro>
-  <xacro:macro name="omni_wheel" params="name parent *origin hq">
+  <xacro:macro name="omni_wheel" params="prefix parent *origin hq">
 <!--WHEEL TIRE -->
     <!-- joint name="joint_${name}_wheel" type="continuous" -->
-    <joint name="joint_${name}_wheel" type="fixed">
+    <joint name="${prefix}wheel_joint" type="fixed">
       <parent link="${parent}"/>
-      <child link="${name}_wheel"/>
-      <insert_block name="origin" />
+      <child link="${prefix}wheel_link"/>
+      <xacro:insert_block name="origin" />
       <axis xyz="0 1 0" rpy="0 0 0" />
       <limit effort="100" velocity="100"/>
       <joint_properties damping="0.0" friction="0.0"/>
     </joint>
-    <link name="${name}_wheel">
+    <link name="${prefix}wheel_link">
       <visual>
         <!-- HIGH RESOLUTION WHEELS -->
@@ -39,16 +40,16 @@
         </xacro:unless>
       </visual>
-      <!-- collision>
+      <collision>
       <origin xyz="0 0 0" rpy="${M_PI/2} 0 0" />
         <geometry>
-          <cylinder length="${omni_wheel_height}" radius="${omni_wheel_radius}" />
+          <cylinder length="0.03" radius="${omni_wheel_radius}" />
         </geometry>
-      </collision -->
-      <collision>
+      </collision>
+      <!--collision>
       <origin xyz="0 0 0" rpy="${M_PI/2} 0 0" />
        <geometry>
          <sphere radius="${omni_wheel_radius}"/>
        </geometry>
-      </collision>
+     </collision-->
       <inertial>
         <mass value="${wheel_mass}" />
@@ -66,12 +67,25 @@
       </actuator>
     </transmission -->
-    <gazebo reference="${name}_wheel">
-			<mu1 value="0.0"/>
-			<mu2 value="0.0"/>
-			<kp value="10000000.0" />
-			<kd value="1.0" />
-			<fdir1 value="1 0 0"/>
-            <turnGravityOff>false</turnGravityOff>
+    <gazebo reference="${prefix}wheel">
+		<mu1 value="0"/>
+		<mu2 value="0"/>
+		<kp value="10000000.0" />
+		<kd value="1.0" />
+		<fdir1 value="1 0 0"/>
+		<material>Gazebo/Black</material>
+		<turnGravityOff>false</turnGravityOff>
     </gazebo>
+    <!--gazebo reference="${name}_wheel">
+		<kp>500000.0</kp>
+		<kd>10.0</kd>
+		<mu1>10</mu1>
+		<mu2>10</mu2>
+		<fdir1>1 0 0</fdir1>
+		<maxVel>1.0</maxVel>
+		<minDepth>0.003</minDepth>
+		<material>Gazebo/Black</material>
+		<turnGravityOff>false</turnGravityOff>
+		<implicitSpringDamper>1</implicitSpringDamper>
+    </gazebo-->
   </xacro:macro>
 </robot>

File: rb1_base_description/urdf/wheels/omni_wheel_v1.urdf.xacro (robot description, xacro)
@@ -3,7 +3,7 @@
   <xacro:property name="M_PI" value="3.1415926535897931" />
   <!-- Wheels -->
-  <property name="omni_wheel_radius" value="0.051" />
-  <property name="omni_wheel_height" value="0.040" />
-  <property name="omni_wheel_mass" value="0.3" /> <!-- in kg-->
+  <xacro:property name="omni_wheel_radius" value="0.051" />
+  <xacro:property name="omni_wheel_height" value="0.040" />
+  <xacro:property name="omni_wheel_mass" value="0.3" /> <!-- in kg-->
   <xacro:macro name="cylinder_inertia" params="m r h">
     <inertia  ixx="${m*(3*r*r+h*h)/12}" ixy = "0" ixz = "0"
@@ -17,5 +17,5 @@
       <parent link="${parent}"/>
       <child link="${name}_wheel"/>
-      <insert_block name="origin" />
+      <xacro:insert_block name="origin" />
       <axis xyz="0 1 0" rpy="0 0 0" />
       <limit effort="100" velocity="100"/>

File: rb1_base_description/urdf/wheels/rubber_wheel.urdf.xacro (robot description, xacro)
@@ -1,46 +1,48 @@
 <?xml version="1.0"?>
 <robot name="wheel" xmlns:xacro="http://www.ros.org/wiki/xacro">
-  <xacro:property name="M_PI" value="3.1415926535897931" />
-  <!-- Wheels -->
-  <property name="wheel_radius" value="0.076" />
-  <property name="wheel_height" value="0.025" />
-  <property name="wheel_mass" value="1.0" /> <!-- in kg-->
-  <xacro:macro name="cylinder_inertia" params="m r h">
-    <inertia  ixx="${m*(3*r*r+h*h)/12}" ixy = "0" ixz = "0"
-              iyy="${m*(3*r*r+h*h)/12}" iyz = "0"
-              izz="${m*r*r/2}" />
-  </xacro:macro>
-  <xacro:macro name="rubber_wheel" params="name parent *origin reflect hq">
-  <!--WHEEL TIRE -->
-    <joint name="joint_${name}_wheel" type="continuous">
-      <parent link="${parent}"/>
-      <child link="${name}_wheel"/>
-      <insert_block name="origin" />
-      <axis xyz="0 1 0" rpy="0 0 0" />
-      <limit effort="100" velocity="100"/>
-      <joint_properties damping="0.0" friction="0.0"/>
-    </joint>
-    <link name="${name}_wheel">
-      <visual>
-        <!-- HIGH RESOLUTION WHEELS -->
-        <xacro:if value="${hq}">
-          <origin xyz="0 0 0" rpy="0 0 0" />
-          <geometry>
-			<xacro:if value="${reflect}">
-				<mesh filename="package://rb1_base_description/meshes/wheels/wheel_rubber_6inch.dae" />
-			</xacro:if>
-			<xacro:unless value="${reflect}">
-				<mesh filename="package://rb1_base_description/meshes/wheels/wheel_rubber_6inch.dae" />
-			</xacro:unless>
-          </geometry>
-        </xacro:if>
-       <!-- LOW RESOLUTION WHEELS -->
-        <xacro:unless value="${hq}">
-          <origin xyz="0 0 0" rpy="${M_PI/2} 0 0" />
-          <geometry>
-            <cylinder length="${wheel_height}" radius="${wheel_radius}" />
-          </geometry>
-        </xacro:unless>
-      </visual>
+	<xacro:include filename="$(find rb1_base_description)/urdf/wheels/rubber_wheel.transmission.xacro"/>
+	<xacro:include filename="$(find rb1_base_description)/urdf/wheels/rubber_wheel.gazebo.xacro"/>
+	<xacro:property name="M_PI" value="3.1415926535897931" />
+	<!-- Wheels -->
+	<xacro:property name="wheel_radius" value="0.076" />
+	<xacro:property name="wheel_height" value="0.025" />
+	<xacro:property name="wheel_mass" value="1.0" /> <!-- in kg-->
+	<xacro:macro name="cylinder_inertia" params="m r h">
+		<inertia	ixx="${m*(3*r*r+h*h)/12}" ixy = "0" ixz = "0"
+					iyy="${m*(3*r*r+h*h)/12}" iyz = "0"
+					izz="${m*r*r/2}" />
+	</xacro:macro>
+	<xacro:macro name="rubber_wheel" params="prefix parent *origin reflect hq">
+	<!--WHEEL TIRE -->
+	<joint name="${prefix}_wheel_joint" type="continuous">
+		<parent link="${parent}"/>
+		<child link="${prefix}_wheel_link"/>
+		<xacro:insert_block name="origin" />
+		<axis xyz="0 1 0" rpy="0 0 0" />
+		<limit effort="100" velocity="100"/>
+		<joint_properties damping="0.0" friction="0.0"/>
+	</joint>
+	<link name="${prefix}_wheel_link">
+		<visual>
+		<!-- HIGH RESOLUTION WHEELS -->
+		<xacro:if value="${hq}">
+			<origin xyz="0 0 0" rpy="0 0 0" />
+			<geometry>
+				<xacro:if value="${reflect}">
+					<mesh filename="package://rb1_base_description/meshes/wheels/wheel_rubber_6inch.dae" />
+				</xacro:if>
+				<xacro:unless value="${reflect}">
+					<mesh filename="package://rb1_base_description/meshes/wheels/wheel_rubber_6inch.dae" />
+				</xacro:unless>
+			</geometry>
+		</xacro:if>
+		<!-- LOW RESOLUTION WHEELS -->
+		<xacro:unless value="${hq}">
+			<origin xyz="0 0 0" rpy="${M_PI/2} 0 0" />
+			<geometry>
+				<cylinder length="${wheel_height}" radius="${wheel_radius}" />
+			</geometry>
+		</xacro:unless>
+		</visual>
       <collision>
 		<origin xyz="0 0 0" rpy="${M_PI/2} 0 0" />
@@ -51,30 +53,10 @@
       <inertial>
         <mass value="${wheel_mass}" />
-        <origin xyz="0 0 0" />
+        <origin xyz="0 0 0" rpy="${M_PI/2} 0 0"/>
         <cylinder_inertia  m="${wheel_mass}" r="${wheel_radius}" h="${wheel_height}" />
       </inertial>
     </link>
-    <!-- Transmission is important to link the joints and the controller (see rb1_control/config/rb1_control.yaml)-->
-    <transmission name="${name}_wheel_joint_trans">
-      <type>transmission_interface/SimpleTransmission</type>
-      <joint name="joint_${name}_wheel">
-          <!-- for the gazebo plugin -->
-          <!-- hardwareInterface>EffortJointInterface</hardwareInterface -->
-          <!-- for ros control controller -->
-          <hardwareInterface>VelocityJointInterface</hardwareInterface>
-      </joint>
-      <actuator name="${name}_wheel_joint_motor">
-        <mechanicalReduction>1</mechanicalReduction>
-        <motorTorqueConstant>20</motorTorqueConstant>
-      </actuator>
-    </transmission>
-    <gazebo reference="${name}_wheel">
-			<mu1 value="5.0"/>
-			<mu2 value="0.5"/>
-			<kp value="10000000.0" />
-			<kd value="1.0" />
-			<fdir1 value="1 0 0"/>
-      <turnGravityOff>false</turnGravityOff>
-    </gazebo>
+	<xacro:rubber_wheel_transmission prefix="${prefix}" />
+	<xacro:rubber_wheel_gazebo prefix="${prefix}" />
   </xacro:macro>
 </robot>
