Commit message: Rebase from 'release/kinetic/rb1_base_description'

File: robots/versions/rb1_base_160721A.urdf.xacro (robot description, xacro)
@@ -1,4 +1,4 @@
 <?xml version="1.0"?>
-<robot name="rb1_base_platform" xmlns:xacro="http://www.ros.org/wiki/xacro">
+<robot name="rb1_base" xmlns:xacro="http://www.ros.org/wiki/xacro">
 	<!-- ***************** -->
 	<!-- Imported elements -->
@@ -6,5 +6,5 @@
 	<!-- First we import all posible elements defined in the urdf.xacro files. All these elements are defined as macro:xacros -->
 	<!-- Import RB1 base elements -->
-    <xacro:include filename="$(find rb1_base_description)/urdf/bases/rb1_base.urdf.xacro" />
+    <xacro:include filename="$(find rb1_base_description)/urdf/bases/rb1_base_v3.urdf.xacro" /> <!-- v3 name from engineering department -->
 	<!-- Import RB1 wheels -->
 	<xacro:include filename="$(find rb1_base_description)/urdf/wheels/rubber_wheel.urdf.xacro" />
@@ -12,4 +12,8 @@
 	<!-- Import all available sensors -->
 	<xacro:include filename="$(find robotnik_sensors)/urdf/all_sensors.urdf.xacro" />
+    <!-- Import Gazebo Stuff -->
+    <xacro:include filename="$(find rb1_base_description)/urdf/common.gazebo.xacro" />
+    <!-- Import Elevator -->
+	<xacro:include filename="$(find rb1_base_description)/urdf/elevator/elevator.urdf.xacro"/>
 	<!-- ***************** -->
 	<!-- Global parameters -->
@@ -18,13 +22,13 @@
 	<!-- Wheel parameters -->
 	<xacro:property name="wheel_offset_x" value="0.0" />    <!-- x,y,z in translation from base_link to the center of the wheel -->
-	<xacro:property name="wheel_offset_y" value="0.217" />
-	<xacro:property name="wheel_offset_z" value="0.051" />
+	<xacro:property name="wheel_offset_y" value="0.218" />
+	<xacro:property name="wheel_offset_z" value="0.0512" />
 	<!-- Castor paramters -->
 	<xacro:property name="omni_back_x" value="0.195" />
 	<xacro:property name="omni_back_y" value="0.0" />
-	<xacro:property name="omni_back_z" value="0.0265" />
-	<xacro:property name="omni_front_x" value="0.133" />
-	<xacro:property name="omni_front_y" value="0.144" />
-	<xacro:property name="omni_front_z" value="0.0265" />
+	<xacro:property name="omni_back_z" value="0.0258" />
+	<xacro:property name="omni_front_x" value="0.132" />
+	<xacro:property name="omni_front_y" value="0.1535" />
+	<xacro:property name="omni_front_z" value="0.0258" />
 	<!-- Flag to select the high or low quality model -->
 	<xacro:property name="hq" value="true" />
@@ -34,43 +38,35 @@
 	<!-- Here we create the robot elements using the xacro:macros imported at the beggining of this file -->
 	<!-- RB-1 base -->
-	<xacro:rb1_base name="rb1_base" publish_bf="true" hq="${hq}" />
-	<!-- Gazebo ros control plugins -->
+	<xacro:rb1_base_v3 prefix="$(arg prefix)" publish_bf="true" hq="${hq}" />
+	<xacro:arg name="prefix" default="rb1_"/>
+	<!-- Gazebo ros control pluggins -->
 	<xacro:ros_control/>
-	<!-- Gazebo skid steering plugins -->
-	<xacro:diff_drive/>
+	<xacro:gazebo_colors prefix="$(arg prefix)"/>
 	<!-- WHEELS -->
-	<xacro:rubber_wheel name="right" parent="base_link" reflect="false" hq="${hq}">
+	<xacro:rubber_wheel prefix="$(arg prefix)right" parent="$(arg prefix)base_link" reflect="false" hq="${hq}">
 		<origin xyz="${wheel_offset_x} -${wheel_offset_y} ${wheel_offset_z}" rpy="0 0 0"/>
 	</xacro:rubber_wheel>
-	<xacro:rubber_wheel name="left" parent="base_link" reflect="true" hq="${hq}">
+	<xacro:rubber_wheel prefix="$(arg prefix)left" parent="$(arg prefix)base_link" reflect="true" hq="${hq}">
 		<origin xyz="${wheel_offset_x} ${wheel_offset_y} ${wheel_offset_z}" rpy="0 0 0"/>
 	</xacro:rubber_wheel>
     <!-- OMNI DIRECTIONAL WHEELS -->
-	<xacro:omni_wheel name="omni_back" parent="base_link" hq="${hq}">
+	<xacro:omni_wheel prefix="$(arg prefix)omni_back" parent="$(arg prefix)base_link" hq="${hq}">
 		<origin xyz="-${omni_back_x} ${omni_back_y} ${omni_back_z}" rpy="0 0 0"/>
 	</xacro:omni_wheel>
-	<xacro:omni_wheel name="omni_front_left" parent="base_link" hq="${hq}">
+	<xacro:omni_wheel prefix="$(arg prefix)omni_front_left" parent="$(arg prefix)base_link" hq="${hq}">
 		<origin xyz="${omni_front_x} ${omni_front_y} ${omni_front_z}" rpy="0 0 0"/>
 	</xacro:omni_wheel>
-	<xacro:omni_wheel name="omni_front_right" parent="base_link" hq="${hq}">
+	<xacro:omni_wheel prefix="$(arg prefix)omni_front_right" parent="$(arg prefix)base_link" hq="${hq}">
 		<origin xyz="${omni_front_x} -${omni_front_y} ${omni_front_z}" rpy="0 0 0"/>
 	</xacro:omni_wheel>
 	<!-- SENSORS -->
-	<!-- xacro:sensor_hokuyo_utm30lx name="hokuyo" parent="base_link">
-		<origin xyz="0.210 0.0 0.305" rpy="0 0 0"/>
-	</xacro:sensor_hokuyo_utm30lx -->
-    <!-- xacro:sensor_hokuyo_urg04lx name="hokuyo" parent="base_link">
-        <origin xyz="0.223 0.0 0.209" rpy="0 3.1416 3.1416"/>
-    </xacro:sensor_hokuyo_urg04lx -->
-	<xacro:sensor_hokuyo_ust10lx name="hokuyo" parent="base_link">
+	<xacro:sensor_hokuyo_ust20lx prefix="$(arg prefix)front_laser" parent="$(arg prefix)base_link">
 		<origin xyz="0.223 0.0 0.159" rpy="0 3.1416 3.1416"/>
-	</xacro:sensor_hokuyo_ust10lx>
-	<xacro:sensor_imu name="imu" parent="base_link">
-		<origin xyz="-0.18 0.0 0.170" rpy="0 0 0"/>
+	</xacro:sensor_hokuyo_ust20lx>
+	<xacro:sensor_imu prefix="$(arg prefix)imu" parent="$(arg prefix)base_link">
+		<origin xyz="0.002 0.053 0.1485" rpy="0 0 0"/>
 	</xacro:sensor_imu>
-<!--
-    <xacro:sensor_kinect name="kinect" parent="base_link">
-        <origin xyz="0.3 0.0 0.16" rpy="0 0 0"/>
-    </xacro:sensor_kinect>
--->
+    <!--xacro:sensor_orbbec_astra prefix="$(arg prefix)front_rgbd_camera" parent="$(arg prefix)base_link">
+        <origin xyz="0.234 0.0125 0.107" rpy="0 0 0"/>
+    </xacro:sensor_orbbec_astra-->
 </robot>

File: robots/versions/rb1_base_171019C.urdf.xacro (robot description, xacro)
@@ -1,4 +1,4 @@
 <?xml version="1.0"?>
-<robot name="rb1_base_platform" xmlns:xacro="http://www.ros.org/wiki/xacro">
+<robot name="rb1_base" xmlns:xacro="http://www.ros.org/wiki/xacro">
 	<!-- ***************** -->
 	<!-- Imported elements -->
@@ -6,5 +6,5 @@
 	<!-- First we import all posible elements defined in the urdf.xacro files. All these elements are defined as macro:xacros -->
 	<!-- Import RB1 base elements -->
-    <xacro:include filename="$(find rb1_base_description)/urdf/bases/rb1_base.urdf.xacro" />
+    <xacro:include filename="$(find rb1_base_description)/urdf/bases/rb1_base_v3.urdf.xacro" /> <!-- v3 name from engineering department -->
 	<!-- Import RB1 wheels -->
 	<xacro:include filename="$(find rb1_base_description)/urdf/wheels/rubber_wheel.urdf.xacro" />
@@ -12,4 +12,8 @@
 	<!-- Import all available sensors -->
 	<xacro:include filename="$(find robotnik_sensors)/urdf/all_sensors.urdf.xacro" />
+    <!-- Import Gazebo Stuff -->
+    <xacro:include filename="$(find rb1_base_description)/urdf/common.gazebo.xacro" />
+    <!-- Import Elevator -->
+	<xacro:include filename="$(find rb1_base_description)/urdf/elevator/elevator.urdf.xacro"/>
 	<!-- ***************** -->
 	<!-- Global parameters -->
@@ -18,13 +22,13 @@
 	<!-- Wheel parameters -->
 	<xacro:property name="wheel_offset_x" value="0.0" />    <!-- x,y,z in translation from base_link to the center of the wheel -->
-	<xacro:property name="wheel_offset_y" value="0.217" />
-	<xacro:property name="wheel_offset_z" value="0.051" />
+	<xacro:property name="wheel_offset_y" value="0.218" />
+	<xacro:property name="wheel_offset_z" value="0.0512" />
 	<!-- Castor paramters -->
 	<xacro:property name="omni_back_x" value="0.195" />
 	<xacro:property name="omni_back_y" value="0.0" />
-	<xacro:property name="omni_back_z" value="0.0265" />
-	<xacro:property name="omni_front_x" value="0.133" />
-	<xacro:property name="omni_front_y" value="0.148" />
-	<xacro:property name="omni_front_z" value="0.0265" />
+	<xacro:property name="omni_back_z" value="0.0270" />
+	<xacro:property name="omni_front_x" value="0.132" />
+	<xacro:property name="omni_front_y" value="0.1535" />
+	<xacro:property name="omni_front_z" value="0.0270" />
 	<!-- Flag to select the high or low quality model -->
 	<xacro:property name="hq" value="true" />
@@ -34,46 +38,35 @@
 	<!-- Here we create the robot elements using the xacro:macros imported at the beggining of this file -->
 	<!-- RB-1 base -->
-	<xacro:rb1_base name="rb1_base" publish_bf="true" hq="${hq}" />
-	<!-- Gazebo ros control plugins -->
+	<xacro:rb1_base_v3 prefix="$(arg prefix)" publish_bf="true" hq="${hq}" />
+	<xacro:arg name="prefix" default="rb1_"/>
+	<!-- Gazebo ros control pluggins -->
 	<xacro:ros_control/>
-	<!-- Gazebo skid steering plugins -->
-	<xacro:diff_drive/>
+	<xacro:gazebo_colors prefix="$(arg prefix)"/>
 	<!-- WHEELS -->
-	<xacro:rubber_wheel name="right" parent="base_link" reflect="false" hq="${hq}">
+	<xacro:rubber_wheel prefix="$(arg prefix)right" parent="$(arg prefix)base_link" reflect="false" hq="${hq}">
 		<origin xyz="${wheel_offset_x} -${wheel_offset_y} ${wheel_offset_z}" rpy="0 0 0"/>
 	</xacro:rubber_wheel>
-	<xacro:rubber_wheel name="left" parent="base_link" reflect="true" hq="${hq}">
+	<xacro:rubber_wheel prefix="$(arg prefix)left" parent="$(arg prefix)base_link" reflect="true" hq="${hq}">
 		<origin xyz="${wheel_offset_x} ${wheel_offset_y} ${wheel_offset_z}" rpy="0 0 0"/>
 	</xacro:rubber_wheel>
     <!-- OMNI DIRECTIONAL WHEELS -->
-	<xacro:omni_wheel name="omni_back" parent="base_link" hq="${hq}">
+	<xacro:omni_wheel prefix="$(arg prefix)omni_back" parent="$(arg prefix)base_link" hq="${hq}">
 		<origin xyz="-${omni_back_x} ${omni_back_y} ${omni_back_z}" rpy="0 0 0"/>
 	</xacro:omni_wheel>
-	<xacro:omni_wheel name="omni_front_left" parent="base_link" hq="${hq}">
+	<xacro:omni_wheel prefix="$(arg prefix)omni_front_left" parent="$(arg prefix)base_link" hq="${hq}">
 		<origin xyz="${omni_front_x} ${omni_front_y} ${omni_front_z}" rpy="0 0 0"/>
 	</xacro:omni_wheel>
-	<xacro:omni_wheel name="omni_front_right" parent="base_link" hq="${hq}">
+	<xacro:omni_wheel prefix="$(arg prefix)omni_front_right" parent="$(arg prefix)base_link" hq="${hq}">
 		<origin xyz="${omni_front_x} -${omni_front_y} ${omni_front_z}" rpy="0 0 0"/>
 	</xacro:omni_wheel>
 	<!-- SENSORS -->
-	<!-- xacro:sensor_hokuyo_utm30lx name="hokuyo" parent="base_link">
-		<origin xyz="0.210 0.0 0.305" rpy="0 0 0"/>
-	</xacro:sensor_hokuyo_utm30lx -->
-    <!-- xacro:sensor_hokuyo_urg04lx name="hokuyo" parent="base_link">
-        <origin xyz="0.223 0.0 0.209" rpy="0 3.1416 3.1416"/>
-    </xacro:sensor_hokuyo_urg04lx -->
-	<xacro:sensor_hokuyo_ust10lx name="hokuyo" parent="base_link">
-		<origin xyz="0.223 0.0 0.159" rpy="0 3.1416 3.1416"/>
-	</xacro:sensor_hokuyo_ust10lx>
-	<xacro:sensor_imu name="imu" parent="base_link">
-		<origin xyz="-0.18 0.0 0.170" rpy="0 0 0"/>
-	</xacro:sensor_imu>
-    <xacro:sensor_orbbec_astra name="orbbec_astra" parent="base_link">
+	<xacro:sensor_sick_tim571 prefix="$(arg prefix)front_laser" parent="$(arg prefix)base_link" prefix_topic="front_laser">
+		<origin xyz="0.219 0.0 0.219" rpy="0 3.1416 3.1416"/>
+	</xacro:sensor_sick_tim571>
+	<xacro:sensor_imu_hector prefix="$(arg prefix)imu" parent="$(arg prefix)base_link">
+		<origin xyz="0.002 0.053 0.1485" rpy="0 0 0"/>
+	</xacro:sensor_imu_hector>
+    <xacro:sensor_orbbec_astra prefix="$(arg prefix)front_rgbd_camera" parent="$(arg prefix)base_link" prefix_topic="front_rgbd_camera">
         <origin xyz="0.234 0.0125 0.107" rpy="0 0 0"/>
     </xacro:sensor_orbbec_astra>
-<!--
-    <xacro:sensor_kinect name="kinect" parent="base_link">
-        <origin xyz="0.3 0.0 0.16" rpy="0 0 0"/>
-    </xacro:sensor_kinect>
--->
 </robot>

File: urdf/bases/rb1_base_v2.urdf.xacro (robot description, xacro)
@@ -1,5 +1,5 @@
 <?xml version="1.0"?>
 <robot name="rb1_base" xmlns:xacro="http://www.ros.org/wiki/xacro">
-  <xacro:macro name="rb1_base" params="prefix publish_bf hq">
+  <xacro:macro name="rb1_base_v2" params="prefix publish_bf hq">
   <!-- Robot mechanical and motor parameters -->
   <xacro:property name="PI" value="3.1415926535897931"/>
@@ -32,5 +32,5 @@
        <xacro:if value="${hq}">
        <geometry>
-         <mesh filename="package://rb1_base_description/meshes/bases/rb1v2_base.dae"/>
+	     <mesh filename="package://rb1_base_description/meshes/bases/rb1v2_base.dae"/>
        </geometry>
        </xacro:if>
@@ -90,8 +90,8 @@
      <origin xyz="0.030 0.000 0.068" rpy="0 0 0 " />
      <parent link="${prefix}front_cover_link"/>
-     <child link="${prefix}base_docking_contact" />
+     <child link="${prefix}base_docking_contact_link" />
   </joint>
-  <!-- FRONT COVER -->
-  <link name="${prefix}base_docking_contact" />
+  <!-- DOCKING LINK -->
+  <link name="${prefix}base_docking_contact_link" />
   </xacro:macro>
 </robot>

File: urdf/bases/rb1_base_v3.urdf.xacro (robot description, xacro)
@@ -1,5 +1,5 @@
 <?xml version="1.0"?>
 <robot name="rb1_base" xmlns:xacro="http://www.ros.org/wiki/xacro">
-  <xacro:macro name="rb1_base" params="prefix publish_bf hq">
+  <xacro:macro name="rb1_base_v3" params="prefix publish_bf hq">
   <!-- Robot mechanical and motor parameters -->
   <xacro:property name="PI" value="3.1415926535897931"/>
@@ -8,10 +8,10 @@
   <xacro:if value="${publish_bf}">
     <link name="${prefix}base_footprint">
-      <visual>
+      <!--visual>
           <origin xyz="0 0 0" rpy="0 0 0" />
           <geometry>
              <box size="0.001 0.001 0.001" />
           </geometry>
-      </visual>
+      </visual-->
     </link>
     <joint name="${prefix}base_footprint_joint" type="fixed">
@@ -32,10 +32,10 @@
        <xacro:if value="${hq}">
        <geometry>
-         <mesh filename="package://rb1_base_description/meshes/bases/rb1v2_base.dae"/>
+	     <mesh filename="package://rb1_base_description/meshes/bases/rb1_base_v3.stl"/>
        </geometry>
        </xacro:if>
        <xacro:unless value="${hq}">
        <geometry>
-       <mesh filename="package://rb1_base_description/meshes/bases/rb1v2_base.stl"/>
+       <mesh filename="package://rb1_base_description/meshes/bases/rb1_base_v3.stl"/>
        </geometry>
        </xacro:unless>
@@ -44,10 +44,10 @@
        </material>
     </visual>
-    <collision>
+    <!--collision>
        <origin xyz="0 0 0" rpy="0 0 0 " />
        <geometry>
-         <mesh filename="package://rb1_base_description/meshes/bases/rb1v2_base.dae"/>
+         <mesh filename="package://rb1_base_description/meshes/bases/rb1_base_v3.dae"/>
        </geometry>
-    </collision>
+    </collision-->
   </link>
   <joint name="${prefix}front_cover_joint" type="fixed">
@@ -67,10 +67,10 @@
        <xacro:if value="${hq}">
        <geometry>
-	     <mesh filename="package://rb1_base_description/meshes/bases/rb1v2_front_cover.dae"/>
+	     <mesh filename="package://rb1_base_description/meshes/bases/rb1_front_cover_v3.stl"/>
        </geometry>
        </xacro:if>
        <xacro:unless value="${hq}">
        <geometry>
-       <mesh filename="package://rb1_base_description/meshes/bases/rb1v2_front_cover.stl"/>
+       <mesh filename="package://rb1_base_description/meshes/bases/rb1_front_cover_v3.stl"/>
        </geometry>
        </xacro:unless>
@@ -82,5 +82,40 @@
        <origin xyz="0 0 0" rpy="0 0 0 " />
        <geometry>
-         <mesh filename="package://rb1_base_description/meshes/bases/rb1v2_front_cover.dae"/>
+         <mesh filename="package://rb1_base_description/meshes/bases/rb1_front_cover_v3.dae"/>
+       </geometry>
+    </collision>
+  </link>
+  <joint name="${prefix}top_covert_joint" type="fixed">
+     <origin xyz="0.0 0.0 0.243" rpy="0 0 0 " />
+     <parent link="${prefix}base_footprint"/>
+     <child link="${prefix}top_cover_link" />
+  </joint>
+  <!-- FRONT COVER -->
+  <link name="${prefix}top_cover_link">
+    <inertial>
+      <mass value="0.25" />
+      <origin xyz="0 0 0" />
+      <inertia  ixx="0.00007" ixy="0.0"  ixz="0.0"  iyy="0.00007"  iyz="0.0"  izz="0.0078" />
+    </inertial>
+    <visual>
+       <origin xyz="0 0 0" rpy="0 0 0" />
+       <xacro:if value="${hq}">
+		   <geometry>
+			 <mesh filename="package://rb1_base_description/meshes/bases/rb1_top_cover_v3.stl"/>
+		   </geometry>
+       </xacro:if>
+       <xacro:unless value="${hq}">
+		   <geometry>
+		   <mesh filename="package://rb1_base_description/meshes/bases/rb1_top_cover_v3.stl"/>
+		   </geometry>
+       </xacro:unless>
+       <material name="black">
+         <color rgba="0.0 0.0 0.0 1"/>
+       </material>
+    </visual>
+    <collision>
+       <origin xyz="0 0 0" rpy="0 0 0 " />
+       <geometry>
+         <mesh filename="package://rb1_base_description/meshes/bases/rb1_top_cover_v3.dae"/>
        </geometry>
     </collision>
@@ -90,8 +125,8 @@
      <origin xyz="0.030 0.000 0.068" rpy="0 0 0 " />
      <parent link="${prefix}front_cover_link"/>
-     <child link="${prefix}base_docking_contact" />
+     <child link="${prefix}base_docking_contact_link" />
   </joint>
-  <!-- FRONT COVER -->
-  <link name="${prefix}base_docking_contact" />
+  <!-- DOCKING LINK -->
+  <link name="${prefix}base_docking_contact_link" />
   </xacro:macro>
 </robot>
